Commit message: исправил небольшие неточности

File: src/mobile_description/urdf/robot_v1.urdf (robot description, URDF)
Before this commit: robot vehicle_blue, 5 links, 4 joints
Joints:
- joint caster_joint: type fixed -> continuous
- joint left_wheel_joint: axis 0 1 0 -> 0 0 1
- joint right_wheel_joint: axis 0 1 0 -> 0 0 1
